File: KiCad/wpt_rx/wpt_rx.kicad_pcb (KiCad board)
At the start: 2 copper layers, 44.4 x 31.8 mm, 28 parts, among them J1 Conn_Coaxial, U1 NCP1117-ADJ_SOT223

Commit message: bump kicad version to 8.0.2, etc.
Parts:
- renumbered RFin1 to TP1, Vfb to TP10, RFin2 to TP2, Vrect to TP3, GND to TP6, Vout to TP7
Connections:
- net Net-(D1-A) renamed /RFin1
- net Net-(D1-K) renamed /Vrect
- net Net-(D2-A) renamed /RFin2
- net Net-(U1-ADJ) renamed /Vfb
Other:
- board text added: "RFin1"
- board text added: "RFin2"
- board text added: "Vfb"
- board text added: "Vrect"
