File: KiCad/wpt_rx/wpt_rx.kicad_sch (KiCad schematic)
At the start: 28 parts, among them J1 Conn_Coaxial, U1 NCP1117-ADJ_SOT223

Commit message: add file exports
Other:
- moved on the sheet: C1, C2, C3, C4, C5, C6, D1, D2, D3, D4, H1, H2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

Commit message: bump kicad version to 8.0.2, etc.
Connections:
- net RFin1: now reaches D1.2 (A), D3.1 (K), J1.2 (Ext), TP1.1
- net Vfb: now reaches R1.1, R2.2, TP10.1, U1.1 (ADJ)
- net Vrect: now reaches C1.1, C3.1, C4.1, D1.1 (K), D2.1 (K), TP3.1, U1.3 (VI)
- net RFin2: now reaches D2.2 (A), D4.1 (K), J1.1 (In), TP2.1
